Commit message: Add files via upload

File: rbt_manipulator/urdf/links_joint.xacro (robot description, xacro)
@@ -1,15 +1,36 @@
 <?xml version="1.0" ?>
 <robot name="mrm" xmlns:xacro="https://www.ros.org/wiki/xacro" >
-	<xacro:macro name="m_joint" params="name type axis_xyz origin_rpy orgin_xyz parent child" >
+	<xacro:macro name="m_joint" params="name type axis_xyz origin_rpy orgin_xyz parent child limit_e limit_l limit_u limit_v" >
 		<joint name="${name}" type="${type}">
 		 <axis xyz="${axis_xyz}" />
-		 <limit effort="1000.0" lower="-3.14" upper="3.14" velocity="0.5" />
+		 <limit effort="${limit_e}" lower="${limit_l}" upper="${limit_u}" velocity="${limit_v}" />
 		 <origin rpy="${origin_rpy}" xyz="${orgin_xyz}" />
 		 <parent link="${parent}" />
 		 <child link="${child}" />
 		</joint>
+		<transmission name="trans_${name}" >
+			<type>transmission_interface/SimpleTransmission</type>
+			<joint name="${name}">
+				<hardwareInterface>hardware_interface/EffortJointInterface</hardwareInterface>
+			</joint>
+			<actuator name="motor_${name}">
+				<hardwareInterface>hardware_interface/EffortJointInterface</hardwareInterface>
+				<mechanicalReduction>1</mechanicalReduction>
+			</actuator>
+		</transmission>
 	</xacro:macro>
-	<xacro:macro name="m_link_cylinder" params="name origin_xyz origin_rpy radius length" >
+	<xacro:macro name="m_link_cylinder" params="name origin_xyz origin_rpy radius length mass ixx ixy ixz iyy iyz izz" >
 		<link name="${name}" >
+			<inertial>
+				<mass value="${mass}" />
+				<origin rpy="${origin_rpy}" xyz="${origin_xyz}" />
+				<inertia ixx="${ixx}" ixy="${ixy}" ixz="${ixz}" iyy="${iyy}" iyz="${iyz}" izz="${izz}" />
+			</inertial>
+			<collision>
+				<origin rpy="${origin_rpy}" xyz="${origin_xyz}" />
+		 		<geometry>
+					<cylinder radius="${radius}" length="${length}" />
+				</geometry>
+			</collision>
 			<visual>
 		 	 <origin rpy="${origin_rpy}" xyz="${origin_xyz}" />
@@ -20,6 +41,17 @@
 		</link>
 	</xacro:macro>
-	<xacro:macro name="m_link_box" params="name origin_xyz origin_rpy size" >
+	<xacro:macro name="m_link_box" params="name origin_xyz origin_rpy size mass ixx ixy ixz iyy iyz izz" >
 		<link name="${name}" >
+			<inertial>
+				<mass value="${mass}" />
+				<origin rpy="${origin_rpy}" xyz="${origin_xyz}" />
+				<inertia ixx="${ixx}" ixy="${ixy}" ixz="${ixz}" iyy="${iyy}" iyz="${iyz}" izz="${izz}" />
+			</inertial>
+			<collision>
+				<origin rpy="${origin_rpy}" xyz="${origin_xyz}" />
+		 	 	<geometry>
+		 			<box size="${size}" />
+	 	 		</geometry>
+			</collision>
 			<visual>
 		 	 <origin rpy="${origin_rpy}" xyz="${origin_xyz}" />
@@ -30,3 +62,25 @@
 		</link>
 	</xacro:macro>
+	<xacro:macro name="m_link_mesh" params="name origin_xyz origin_rpy meshfile meshscale mass ixx ixy ixz iyy iyz izz" >
+		<link name="${name}" >
+			<inertial>
+				<mass value="${mass}" />
+				<origin rpy="${origin_rpy}" xyz="${origin_xyz}" />
+				<inertia ixx="${ixx}" ixy="${ixy}" ixz="${ixz}" iyy="${iyy}" iyz="${iyz}" izz="${izz}" />
+			</inertial>
+			<collision>
+				<origin rpy="${origin_rpy}" xyz="${origin_xyz}" />
+		 	 	<geometry>
+		 			<mesh filename="${meshfile}" scale="${meshscale}" />
+	 	 		</geometry>
+			</collision>
+			<visual>
+		 	 <origin rpy="${origin_rpy}" xyz="${origin_xyz}" />
+		 	 <geometry>
+		 		<mesh filename="${meshfile}" scale="${meshscale}" />
+	 	 	 </geometry>
+	 	 	 <material name="light_black" />
+ 	 		</visual>
+		</link>
+	</xacro:macro>
 </robot>

File: rbt_manipulator/urdf/mrm.xacro (robot description, xacro)
@@ -6,15 +6,20 @@
 	<!-- END Include -->
 	<!-- BGN Robot description -->
-	<xacro:m_link_box name="${l00}" origin_xyz="0 0 0" origin_rpy="0 0 0" size="1 1 1" />
-	<xacro:m_joint name="${l00}__${l01}" type="revolute" axis_xyz="0 0 1" origin_rpy="0 0 0" orgin_xyz="0 0 0.5" parent="${l00}" child="${l01}" />
-	<xacro:m_link_cylinder name="${l01}" origin_xyz="0 0 0.2" origin_rpy="0 0 0" radius="0.35" length="0.4" />
-	<xacro:m_joint name="${l01}__${l02}" type="revolute" axis_xyz="0 1 0" origin_rpy="0 0 0" orgin_xyz="0 0 0.4" parent="${l01}" child="${l02}" />
-	<xacro:m_link_cylinder name="${l02}" origin_xyz="0 0 0.4" origin_rpy="0 0 0" radius="0.15" length="0.8" />
-	<xacro:m_joint name="${l02}__${l03}" type="revolute" axis_xyz="0 1 0" origin_rpy="0 0 0" orgin_xyz="0 0 0.8" parent="${l02}" child="${l03}" />
-	<xacro:m_link_cylinder name="${l03}" origin_xyz="0 0 0.4" origin_rpy="0 0 0" radius="0.15" length="0.8" />
-	<xacro:m_joint name="${l03}__${l04}" type="revolute" axis_xyz="0 1 0" origin_rpy="0 0 0" orgin_xyz="0 0 0.8" parent="${l03}" child="${l04}" />
-	<xacro:m_link_cylinder name="${l04}" origin_xyz="0 0 0.4" origin_rpy="0 0 0" radius="0.15" length="0.8" />
-	<xacro:m_joint name="${l04}__${l05}" type="revolute" axis_xyz="0 0 1" origin_rpy="0 0 0" orgin_xyz="0 0 0.8" parent="${l04}" child="${l05}" />
-	<xacro:m_link_cylinder name="${l05}" origin_xyz="0 0 0.125" origin_rpy="0 0 0" radius="0.15" length="0.25" />
+	<xacro:m_link_box name="${l00}" origin_xyz="0 0 0" origin_rpy="0 0 0" mass="1024" ixx="170.6667" ixy="0" ixz="0" iyy="170.6667" iyz="0" izz="170.6667" size="1 1 1" />
+	<xacro:m_joint name="${l00}__${l01}" type="revolute" axis_xyz="0 0 1" origin_rpy="0 0 0" orgin_xyz="0 0 0.5" parent="${l00}" child="${l01}" limit_e="1000.0" limit_l="-3.14" limit_u="3.14" limit_v="0.5"/>
+	<xacro:m_link_cylinder name="${l01}" origin_xyz="0 0 0.2" origin_rpy="0 0 0" mass="57.906" ixx="12.679" ixy="0" ixz="0" iyy="12.679" iyz="0" izz="0.651" radius="0.35" length="0.4" />
+	<xacro:m_joint name="${l01}__${l02}" type="revolute" axis_xyz="0 1 0" origin_rpy="0 0 0" orgin_xyz="0 0 0.4" parent="${l01}" child="${l02}"  limit_e="1000.0" limit_l="0" limit_u="0.5" limit_v="0.5"/>
+	<xacro:m_link_cylinder name="${l02}" origin_xyz="0 0 0.4" origin_rpy="0 0 0" mass="57.906" ixx="12.679" ixy="0" ixz="0" iyy="12.679" iyz="0" izz="0.651" radius="0.15" length="0.8" />
+	<xacro:m_joint name="${l02}__${l03}" type="revolute" axis_xyz="0 1 0" origin_rpy="0 0 0" orgin_xyz="0 0 0.8" parent="${l02}" child="${l03}"  limit_e="1000.0" limit_l="0" limit_u="0.75" limit_v="0.5"/>
+	<xacro:m_link_cylinder name="${l03}" origin_xyz="0 0 0.4" origin_rpy="0 0 0" mass="57.906" ixx="12.679" ixy="0" ixz="0" iyy="12.679" iyz="0" izz="0.651" radius="0.15" length="0.8" />
+	<xacro:m_joint name="${l03}__${l04}" type="revolute" axis_xyz="0 1 0" origin_rpy="0 0 0" orgin_xyz="0 0 0.8" parent="${l03}" child="${l04}"  limit_e="1000.0" limit_l="0" limit_u="0.75" limit_v="0.5"/>
+	<xacro:m_link_cylinder name="${l04}" origin_xyz="0 0 0.4" origin_rpy="0 0 0" mass="57.906" ixx="12.679" ixy="0" ixz="0" iyy="12.679" iyz="0" izz="0.651" radius="0.15" length="0.8" />
+	<xacro:m_joint name="${l04}__${l05}" type="revolute" axis_xyz="0 0 1" origin_rpy="0 0 0" orgin_xyz="0 0 0.8" parent="${l04}" child="${l05}"  limit_e="1000.0" limit_l="-3.14" limit_u="3.14" limit_v="0.5"/>
+	<xacro:m_link_cylinder name="${l05}" origin_xyz="0 0 0.125" origin_rpy="0 0 0" mass="18.056" ixx="0.479" ixy="0" ixz="0" iyy="0.479" iyz="0" izz="0.204" radius="0.15" length="0.25" />
     <!-- END Robot description -->
+    <gazebo>
+    	<plugin name="gazebo_ros_control" filename="libgazebo_ros_control.so">
+    		<robotNamespace>/mrm</robotNamespace>
+    	</plugin>
+    </gazebo>
 </robot>

Commit message: Add files via upload

File: rbt_manipulator/urdf/links_joint.xacro (robot description, xacro)
@@ -20,5 +20,5 @@
 		</transmission>
 	</xacro:macro>
-	<xacro:macro name="m_link_cylinder" params="name origin_xyz origin_rpy radius length mass ixx ixy ixz iyy iyz izz" >
+	<xacro:macro name="m_link_cylinder" params="name origin_xyz origin_rpy radius length mass ixx ixy ixz iyy iyz izz color_c rgba" >
 		<link name="${name}" >
 			<inertial>
@@ -38,8 +38,11 @@
 		 		<cylinder radius="${radius}" length="${length}" />
 	 	 	 </geometry>
+	 	 	 <material name="${color_c}">
+	 			<color rgba="${rgba}" />
+	 		</material>
  	 		</visual>
 		</link>
 	</xacro:macro>
-	<xacro:macro name="m_link_box" params="name origin_xyz origin_rpy size mass ixx ixy ixz iyy iyz izz" >
+	<xacro:macro name="m_link_box" params="name origin_xyz origin_rpy size mass ixx ixy ixz iyy iyz izz color_c rgba" >
 		<link name="${name}" >
 			<inertial>
@@ -59,4 +62,7 @@
 		 		<box size="${size}" />
 	 	 	 </geometry>
+	 	 	 <material name="${color_c}">
+	 			<color rgba="${rgba}" />
+	 		</material>
  	 		</visual>
 		</link>

File: rbt_manipulator/urdf/mrm.xacro (robot description, xacro)
@@ -6,15 +6,15 @@
 	<!-- END Include -->
 	<!-- BGN Robot description -->
-	<xacro:m_link_box name="${l00}" origin_xyz="0 0 0" origin_rpy="0 0 0" mass="1024" ixx="170.6667" ixy="0" ixz="0" iyy="170.6667" iyz="0" izz="170.6667" size="1 1 1" />
+	<xacro:m_link_box name="${l00}" origin_xyz="0 0 0" origin_rpy="0 0 0" mass="1024" ixx="170.6667" ixy="0" ixz="0" iyy="170.6667" iyz="0" izz="170.6667" size="1 1 1" color_c="Black" rgba="0 0 0 1.0"/>
 	<xacro:m_joint name="${l00}__${l01}" type="revolute" axis_xyz="0 0 1" origin_rpy="0 0 0" orgin_xyz="0 0 0.5" parent="${l00}" child="${l01}" limit_e="1000.0" limit_l="-3.14" limit_u="3.14" limit_v="0.5"/>
-	<xacro:m_link_cylinder name="${l01}" origin_xyz="0 0 0.2" origin_rpy="0 0 0" mass="57.906" ixx="12.679" ixy="0" ixz="0" iyy="12.679" iyz="0" izz="0.651" radius="0.35" length="0.4" />
-	<xacro:m_joint name="${l01}__${l02}" type="revolute" axis_xyz="0 1 0" origin_rpy="0 0 0" orgin_xyz="0 0 0.4" parent="${l01}" child="${l02}"  limit_e="1000.0" limit_l="0" limit_u="0.5" limit_v="0.5"/>
-	<xacro:m_link_cylinder name="${l02}" origin_xyz="0 0 0.4" origin_rpy="0 0 0" mass="57.906" ixx="12.679" ixy="0" ixz="0" iyy="12.679" iyz="0" izz="0.651" radius="0.15" length="0.8" />
-	<xacro:m_joint name="${l02}__${l03}" type="revolute" axis_xyz="0 1 0" origin_rpy="0 0 0" orgin_xyz="0 0 0.8" parent="${l02}" child="${l03}"  limit_e="1000.0" limit_l="0" limit_u="0.75" limit_v="0.5"/>
-	<xacro:m_link_cylinder name="${l03}" origin_xyz="0 0 0.4" origin_rpy="0 0 0" mass="57.906" ixx="12.679" ixy="0" ixz="0" iyy="12.679" iyz="0" izz="0.651" radius="0.15" length="0.8" />
-	<xacro:m_joint name="${l03}__${l04}" type="revolute" axis_xyz="0 1 0" origin_rpy="0 0 0" orgin_xyz="0 0 0.8" parent="${l03}" child="${l04}"  limit_e="1000.0" limit_l="0" limit_u="0.75" limit_v="0.5"/>
-	<xacro:m_link_cylinder name="${l04}" origin_xyz="0 0 0.4" origin_rpy="0 0 0" mass="57.906" ixx="12.679" ixy="0" ixz="0" iyy="12.679" iyz="0" izz="0.651" radius="0.15" length="0.8" />
+	<xacro:m_link_cylinder name="${l01}" origin_xyz="0 0 0.2" origin_rpy="0 0 0" mass="57.906" ixx="12.679" ixy="0" ixz="0" iyy="12.679" iyz="0" izz="0.651" radius="0.35" length="0.4" color_c="Red_d" rgba="0.4 0 0 1.0" />
+	<xacro:m_joint name="${l01}__${l02}" type="revolute" axis_xyz="0 1 0" origin_rpy="0 0 0" orgin_xyz="0 0 0.4" parent="${l01}" child="${l02}"  limit_e="1000.0" limit_l="0" limit_u="1.5" limit_v="0.5"/>
+	<xacro:m_link_cylinder name="${l02}" origin_xyz="0 0 0.4" origin_rpy="0 0 0" mass="57.906" ixx="12.679" ixy="0" ixz="0" iyy="12.679" iyz="0" izz="0.651" radius="0.15" length="0.8" color_c="Red_d1" rgba="0.6 0 0 1.0" />
+	<xacro:m_joint name="${l02}__${l03}" type="revolute" axis_xyz="0 1 0" origin_rpy="0 0 0" orgin_xyz="0 0 0.8" parent="${l02}" child="${l03}"  limit_e="1000.0" limit_l="-1.57" limit_u="1.57" limit_v="0.5"/>
+	<xacro:m_link_cylinder name="${l03}" origin_xyz="0 0 0.4" origin_rpy="0 0 0" mass="57.906" ixx="12.679" ixy="0" ixz="0" iyy="12.679" iyz="0" izz="0.651" radius="0.15" length="0.8" color_c="Red_d2" rgba="1.0 0 0 1.0" />
+	<xacro:m_joint name="${l03}__${l04}" type="revolute" axis_xyz="0 1 0" origin_rpy="0 0 0" orgin_xyz="0 0 0.8" parent="${l03}" child="${l04}"  limit_e="1000.0" limit_l="-1.4" limit_u="1.8" limit_v="0.5"/>
+	<xacro:m_link_cylinder name="${l04}" origin_xyz="0 0 0.4" origin_rpy="0 0 0" mass="57.906" ixx="12.679" ixy="0" ixz="0" iyy="12.679" iyz="0" izz="0.651" radius="0.15" length="0.8" color_c="Red_l" rgba="1.0 0.2 0.2 1.0" />
 	<xacro:m_joint name="${l04}__${l05}" type="revolute" axis_xyz="0 0 1" origin_rpy="0 0 0" orgin_xyz="0 0 0.8" parent="${l04}" child="${l05}"  limit_e="1000.0" limit_l="-3.14" limit_u="3.14" limit_v="0.5"/>
-	<xacro:m_link_cylinder name="${l05}" origin_xyz="0 0 0.125" origin_rpy="0 0 0" mass="18.056" ixx="0.479" ixy="0" ixz="0" iyy="0.479" iyz="0" izz="0.204" radius="0.15" length="0.25" />
+	<xacro:m_link_box name="${l05}" origin_xyz="0 0 0" origin_rpy="0 0 0" mass="18.056" ixx="0.479" ixy="0" ixz="0" iyy="0.479" iyz="0" izz="0.204" size="3.0 3.0 0.15" color_c="White" rgba="1.0 1.0 1.0 1.0" />
     <!-- END Robot description -->
     <gazebo>
